Commit message: changes in xacro and package.xml

File: urdf/robotont_realsense.urdf.xacro (robot description, xacro)
@@ -3,3 +3,29 @@
 	<xacro:include filename="$(find robotont_nuc_description)/urdf/_d435.urdf.xacro"/>
     <xacro:include filename="$(find robotont_description)/urdf/robotont_base.urdf.xacro"/>
+    <xacro:sensor_d435 parent="${prefix}base_link" prefix="${prefix}">
+        <origin xyz="-0.12 0 0.21" rpy="0 0 0"/>
+    </xacro:sensor_d435>
+    <!-- Computer -->
+    <link name="${prefix}computer_link">
+        <visual>
+            <geometry>
+                <box size="0.11 0.11 0.04"/>
+            </geometry>
+            <origin rpy="0 0 0" xyz="0 0 0"/>
+            <material name="computer_material">
+                <color rgba="0.1 0.1 0.1 1"/>
+            </material>
+        </visual>
+    </link>
+    <joint
+		name="${prefix}computer_joint"
+		type="fixed"
+	>
+        <parent link="${prefix}base_link" />
+        <child link="${prefix}computer_link" />
+        <origin
+			xyz="-0.01 0 0.085"
+			rpy="0 0 0"
+		/>
+    </joint>
 </robot>

Commit message: removed _d435.urdf.xacro, two launch files, modified package.xml and robotont_realsense.urdf.xacro

File: urdf/robotont_realsense.urdf.xacro (robot description, xacro)
@@ -1,7 +1,8 @@
 <?xml version="1.0"?>
 <robot xmlns:xacro="http://ros.org/wiki/xacro" name="robotont">
-	<xacro:include filename="$(find robotont_nuc_description)/urdf/_d435.urdf.xacro"/>
+	<xacro:include filename="$(find realsense2_description)/urdf/_d435.urdf.xacro" />
     <xacro:include filename="$(find robotont_description)/urdf/robotont_base.urdf.xacro"/>
-    <xacro:sensor_d435 parent="${prefix}base_link" prefix="${prefix}">
+    <xacro:property name= "prefix" value="$(arg prefix)"/>
+    <xacro:sensor_d435 parent="${prefix}base_link">
         <origin xyz="-0.12 0 0.21" rpy="0 0 0"/>
     </xacro:sensor_d435>

Commit message: added collision tag to computer_link

File: urdf/robotont_realsense.urdf.xacro (robot description, xacro)
@@ -18,15 +18,15 @@
             </material>
         </visual>
+        <collision>
+            <geometry>
+                <box size="0.11 0.11 0.04"/>
+            </geometry>
+            <origin rpy="0 0 0" xyz="0 0 0"/>
+        </collision>
     </link>
-    <joint
-		name="${prefix}computer_joint"
-		type="fixed"
-	>
-        <parent link="${prefix}base_link" />
-        <child link="${prefix}computer_link" />
-        <origin
-			xyz="-0.01 0 0.085"
-			rpy="0 0 0"
-		/>
+    <joint name="${prefix}computer_joint" type="fixed">
+        <parent link="${prefix}base_link"/>
+        <child link="${prefix}computer_link"/>
+        <origin xyz="-0.01 0 0.085" rpy="0 0 0"/>
     </joint>
 </robot>

Commit message: added if to xacro

File: urdf/robotont_realsense.urdf.xacro (robot description, xacro)
@@ -1,11 +1,19 @@
 <?xml version="1.0"?>
 <robot xmlns:xacro="http://ros.org/wiki/xacro" name="robotont">
-    <xacro:include filename="$(find realsense2_description)/urdf/_d435.urdf.xacro" />
+	<xacro:include filename="$(find realsense2_description)/urdf/_d435.urdf.xacro" />
     <xacro:include filename="$(find robotont_description)/urdf/robotont_base.urdf.xacro"/>
     <xacro:arg name= "add_plug" default="false"/>
+    <xacro:arg name= "simulated" default="false"/>
     <xacro:property name= "prefix" value="$(arg prefix)"/>
-    <xacro:sensor_d435 parent="${prefix}base_link" use_nominal_extrinsics="false">
-        <origin xyz="-0.12 0 0.21" rpy="0 0 0"/>
-    </xacro:sensor_d435>
+    <xacro:if value="$(arg simulated)">
+        <xacro:sensor_d435 parent="${prefix}base_link" use_nominal_extrinsics="true">
+            <origin xyz="-0.12 0 0.21" rpy="0 0 0"/>
+        </xacro:sensor_d435>
+    </xacro:if>
+    <xacro:unless value="$(arg simulated)">
+        <xacro:sensor_d435 parent="${prefix}base_link" use_nominal_extrinsics="false">
+            <origin xyz="-0.12 0 0.21" rpy="0 0 0"/>
+        </xacro:sensor_d435>
+    </xacro:unless>
     <!-- Computer -->
     <link name="${prefix}computer_link">

Commit message: separated camera assembly

File: urdf/robotont_realsense.urdf.xacro (robot description, xacro)
@@ -6,12 +6,44 @@
     <xacro:arg name= "simulated" default="false"/>
     <xacro:property name= "prefix" value="$(arg prefix)"/>
+    <!-- Camera assembly -->
+    <link name="${prefix}camera_assembly_link1">
+        <visual>
+            <geometry>
+                <mesh scale="0.001 0.001 0.001" filename="package://robotont_nuc_description/meshes/camera_assembly_part1.stl"/>
+            </geometry>
+            <material name="frame_material">
+                <color rgba="1 1 1 1"/>
+            </material>
+        </visual>
+    </link>
+    <joint name="${prefix}camera_assembly_joint1" type="fixed">
+        <parent link="${prefix}base_footprint"/>
+        <child link="${prefix}camera_assembly_link1"/>
+        <origin xyz="0 0 0.0125" rpy="0 0 ${pi/2}"/>
+    </joint>
+    <link name="${prefix}camera_assembly_link2">
+        <visual>
+            <geometry>
+                <mesh scale="0.001 0.001 0.001" filename="package://robotont_nuc_description/meshes/camera_assembly_part2.stl"/>
+            </geometry>
+            <material name="base_material">
+                <color rgba="1 1 1 0.8"/>
+            </material>
+        </visual>
+    </link>
+    <joint name="${prefix}camera_assembly_joint2" type="fixed">
+        <parent link="${prefix}base_footprint"/>
+        <child link="${prefix}camera_assembly_link2"/>
+        <origin xyz="0 0 0.0125" rpy="0 0 ${pi/2}"/>
+    </joint>
+    <!-- Realsense -->
     <xacro:if value="$(arg simulated)">
         <xacro:sensor_d435 parent="${prefix}base_link" use_nominal_extrinsics="true">
-            <origin xyz="-0.12 0 0.21" rpy="0 0 0"/>
+            <origin xyz="-0.115 0 0.2025" rpy="0 0 0"/>
         </xacro:sensor_d435>
     </xacro:if>
     <xacro:unless value="$(arg simulated)">
         <xacro:sensor_d435 parent="${prefix}base_link" use_nominal_extrinsics="false">
-            <origin xyz="-0.12 0 0.21" rpy="0 0 0"/>
+            <origin xyz="-0.115 0 0.2025" rpy="0 0 0"/>
         </xacro:sensor_d435>
     </xacro:unless>

Commit message: ns

File: urdf/robotont_realsense.urdf.xacro (robot description, xacro)
@@ -5,5 +5,4 @@
     <xacro:arg name= "add_plug" default="false"/>
     <xacro:arg name= "simulated" default="false"/>
-    <xacro:property name= "prefix" value="$(arg prefix)"/>
     <!-- Camera assembly -->
     <link name="${prefix}camera_assembly_link1">
@@ -39,10 +38,10 @@
     <!-- Realsense -->
     <xacro:if value="$(arg simulated)">
-        <xacro:sensor_d435 parent="${prefix}base_link" use_nominal_extrinsics="true">
+        <xacro:sensor_d435 name="${prefix}camera" parent="${prefix}base_link" use_nominal_extrinsics="true">
             <origin xyz="-0.115 0 0.2025" rpy="0 0 0"/>
         </xacro:sensor_d435>
     </xacro:if>
     <xacro:unless value="$(arg simulated)">
-        <xacro:sensor_d435 parent="${prefix}base_link" use_nominal_extrinsics="false">
+        <xacro:sensor_d435 name="${prefix}camera" parent="${prefix}base_link" use_nominal_extrinsics="false">
             <origin xyz="-0.115 0 0.2025" rpy="0 0 0"/>
         </xacro:sensor_d435>
