Commit message: robotont_nuc_description - Make model compatible with gz sim 8

File: urdf/gen2_1/camera.urdf.xacro (robot description, xacro)
@@ -10,5 +10,5 @@
             <visual>
                 <geometry>
-                    <mesh filename="package://robotont_nuc_description/meshes/gen2_1/camera_assembly_part1.STL"/>
+                    <mesh filename="file://$(find robotont_nuc_description)/meshes/gen2_1/camera_assembly_part1.STL"/>
                 </geometry>
                 <material name="camera_frame_material">
@@ -25,5 +25,5 @@
             <visual>
                 <geometry>
-                    <mesh filename="package://robotont_nuc_description/meshes/gen2_1/camera_assembly_part2.STL"/>
+                    <mesh filename="file://$(find robotont_nuc_description)/meshes/gen2_1/camera_assembly_part2.STL"/>
                 </geometry>
                 <material name="camera_base_material">

File: urdf/gen2_1/nuc.urdf.xacro (robot description, xacro)
@@ -11,5 +11,5 @@
             <visual>
                 <geometry>
-                    <mesh filename="package://robotont_nuc_description/meshes/gen2_1/payload_tray.STL"/>
+                    <mesh filename="file://$(find robotont_nuc_description)/meshes/gen2_1/payload_tray.STL"/>
                 </geometry>
                 <material name="nuc_frame_material">
@@ -35,5 +35,5 @@
             <visual>
                 <geometry>
-                    <mesh filename="package://robotont_nuc_description/meshes/shared/NUC12WSK.STL"/>
+                    <mesh filename="file://$(find robotont_nuc_description)/meshes/shared/NUC12WSK.STL"/>
                 </geometry>
                 <material name="nuc_material">

File: urdf/gen3/camera.urdf.xacro (robot description, xacro)
@@ -13,5 +13,5 @@
             <visual>
                 <geometry>
-                    <mesh filename="package://robotont_nuc_description/meshes/gen3/camera_module.STL"/>
+                    <mesh filename="file://$(find robotont_nuc_description)/meshes/gen3/camera_module.STL"/>
                 </geometry>
                 <material name="camera_mount_material">

File: urdf/gen3/nuc.urdf.xacro (robot description, xacro)
@@ -11,5 +11,5 @@
             <visual>
                 <geometry>
-                    <mesh filename="package://robotont_nuc_description/meshes/gen3/payload_tray.STL"/>
+                    <mesh filename="file://$(find robotont_nuc_description)/meshes/gen3/payload_tray.STL"/>
                 </geometry>
                 <material name="nuc_frame_material">
@@ -36,5 +36,5 @@
                 <origin xyz="0 0 -0.006"/>
                 <geometry>
-                    <mesh filename="package://robotont_nuc_description/meshes/shared/NUC12WSK.STL"/>
+                    <mesh filename="file://$(find robotont_nuc_description)/meshes/shared/NUC12WSK.STL"/>
                 </geometry>
                 <material name="nuc_material">

File: urdf/gen3/robotont_realsense.urdf.xacro (robot description, xacro)
@@ -1,10 +1,9 @@
 <?xml version="1.0"?>
 <robot xmlns:xacro="http://ros.org/wiki/xacro" name="robotont">
-    <xacro:include filename="$(find realsense2_description)/urdf/_d435i.urdf.xacro" />
+    <xacro:include filename="$(find realsense2_description)/urdf/_d435i.urdf.xacro"/>
     <xacro:include filename="$(find robotont_description)/urdf/gen3/robotont.urdf.xacro"/>
     <xacro:include filename="$(find robotont_nuc_description)/urdf/gen3/camera.urdf.xacro"/>
     <xacro:include filename="$(find robotont_nuc_description)/urdf/gen3/nuc.urdf.xacro"/>
-    <xacro:arg name= "add_plug" default="false"/>
-    <xacro:arg name= "simulated" default="false"/>
+    <xacro:arg name="simulated" default="false"/>
     <xacro:property name="frame_height" value="0.065"/>
     <xacro:property name="frame_ground_clearance" value="0.014"/>
@@ -13,12 +12,12 @@
     <!-- Camera assembly -->
     <xacro:camera_macro
-        color="${camera_mount_color}"
-        frame_height="${frame_height}"
-        frame_ground_clearance="${frame_ground_clearance}"
-        prefix="${prefix}"
+            color="${camera_mount_color}"
+            frame_height="${frame_height}"
+            frame_ground_clearance="${frame_ground_clearance}"
+            prefix="${prefix}"
     />
     <!-- Realsense -->
     <xacro:if value="$(arg simulated)">
-        <xacro:sensor_d435i name="${prefix}camera" parent="${prefix}" use_nominal_extrinsics="true">
+        <xacro:sensor_d435i name="${prefix}camera" parent="${prefix}base_link" use_nominal_extrinsics="true">
             <origin xyz="-0.105 0 0.197" rpy="0 0 0"/>
         </xacro:sensor_d435i>
@@ -31,8 +30,8 @@
     <!-- NUC -->
     <xacro:nuc_macro
-        color="${nuc_frame_color}"
-        frame_height="${frame_height}"
-        frame_ground_clearance="${frame_ground_clearance}"
-        prefix="${prefix}"
+            color="${nuc_frame_color}"
+            frame_height="${frame_height}"
+            frame_ground_clearance="${frame_ground_clearance}"
+            prefix="${prefix}"
     />
 </robot>
